File: Flexible-Determinist/output/pcbs/flexible-determinist.kicad_pcb (KiCad board)
At the start: 2 copper layers, 234.5 x 118.6 mm, 74 parts

Commit message: add mounting holes
Parts:
- added _3: , MountingHole_2.2mm_M2_Pad_Via, F.Cu at (98.3, 130.4)
- added _4: , MountingHole_2.2mm_M2_Pad_Via, F.Cu at (128.9, 177.6)
- added _5: , MountingHole_2.2mm_M2_Pad_Via, F.Cu at (162.3, 104.2)
- added _6: , MountingHole_2.2mm_M2_Pad_Via, F.Cu at (246.4, 86.7)
- added _7: , MountingHole_2.2mm_M2_Pad_Via, F.Cu at (226.3, 130.4)
- added _8: , MountingHole_2.2mm_M2_Pad_Via, F.Cu at (195.8, 177.6)
- _1: footprint MountingHole_2.2mm_M2_Pad_Via -> Feather_RP2040
- _2: footprint Feather_nRF52840 -> MountingHole_2.2mm_M2_Pad_Via
- moved _1 107.3 mm to (162.3, 141.2), turned to -90 degrees
- moved _2 100.2 mm to (78.2, 86.7), turned to -10 degrees
Connections:
- _1 pad 1: (no net) -> VBAT
- _2 pad 1: VBAT -> (no net)
